File: cellular-featherwing-pcb.kicad_pcb (KiCad board)
At the start: 2 copper layers, 54 x 28 mm, 69 parts, among them J1 SIM8060-6-0-14-00-A, J2 TSM-116-01-L-SV, J3 TSM-112-01-L-SV, J4 U.FL-R-SMT, U1 BG96, U2 TPS63020QDSJTQ1, U3 TXB0108DQSR, U4 MAX8868EUK30+T

Commit message: Clean DRC
Routing:
- net VBAT_RF: track 12.1 -> 18.4 mm
- net 3V3: track 37.0 -> 36.0 mm
- net (no net): track 1.41 -> 0.45 mm
- net Net-(C1-Pad1): track 20.4 -> 21.3 mm
- net GND: track 43.1 -> 42.3 mm
- removed copper zone on B.Cu, net Net-(C1-Pad1)
Changed lines of the file:
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@@
     (property "Sheetname" "")
     (attr through_hole)
-    (fp_text reference "J1" (at -2.427355 -8.743475 180) (layer "F.SilkS")
+    (fp_text reference "J1" (at -2.427355 -8.743475 180) (layer "F.SilkS") hide
       (effects (font (size 1.000969 1.000969) (thickness 0.15)))
     )
@@
   )
   (gr_rect locked (start 121 109) (end 175 81) (layer "Edge.Cuts") (width 0.1) (fill none))
-  (segment (start 147.9 83.52) (end 147.9 83.1384) (width 0.25) (layer "F.Cu") (net 0))
   (segment (start 166.33 93.25) (end 165.8808 93.25) (width 0.25) (layer "F.Cu") (net 0))
-  (segment (start 165.7552 98.75) (end 166.33 98.75) (width 0.25) (layer "F.Cu") (net 0))
   (segment (start 153.5 104.6) (end 152.4 104.6) (width 0.2) (layer "F.Cu") (net 15))
   (segment (start 149.3 106.2755) (end 149.7 106.6755) (width 0.2) (layer "F.Cu") (net 15))
@@
   (segment (start 134.38 100.1154) (end 134.38 99.72) (width 0.2) (layer "F.Cu") (net 15))
   (segment (start 150.1245 107.1) (end 149.7 106.6755) (width 0.2) (layer "F.Cu") (net 15))
-  (segment (start 142.6625 105.9) (end 142.6625 106.5691) (width 0.2) (layer "F.Cu") (net 15))
   (segment (start 154.15 100.8) (end 154.2 100.85) (width 0.2) (layer "F.Cu") (net 15))
   (segment (start 134.8232 100.5586) (end 134.38 100.1154) (width 0.2) (layer "F.Cu") (net 15))
@@
   (segment (start 166.48 90.6188) (end 166.48 89.9) (width 0.2) (layer "B.Cu") (net 15))
   (segment (start 152.3524 92.8624) (end 151.7396 92.8624) (width 0.2) (layer "B.Cu") (net 15))
-  (segment (start 138.9888 93.345) (end 138.8872 93.345) (width 0.2) (layer "B.Cu") (net 15))
   (segment (start 143.6142 93.6244) (end 143.6142 93.3984) (width 0.2) (layer "B.Cu") (net 15))
   (segment (start 142.748 92.5322) (end 140.8684 92.5322) (width 0.2) (layer "B.Cu") (net 15))
@@
   (segment (start 148.9756 92.1256) (end 149.55 92.7) (width 0.2) (layer "B.Cu") (net 27))
   (segment (start 149.55 93.35) (end 149.8 93.6) (width 0.2) (layer "B.Cu") (net 27))
-  (segment (start 144.3 95.5) (end 144.3 96.2) (width 0.2) (layer "B.Cu") (net 27))
   (segment (start 144.3 95.5) (end 144.3 93.8986) (width 0.2) (layer "B.Cu") (net 27))
   (segment (start 145.2244 92.1256) (end 148.9756 92.1256) (width 0.2) (layer "B.Cu") (net 27))
@@
   (segment (start 159.1 100.6) (end 161.998685 100.6) (width 0.2) (layer "B.Cu") (net 27))
   (segment (start 144.5742 92.7758) (end 145.2244 92.1256) (width 0.2) (layer "B.Cu") (net 27))
-  (segment (start 144.3 96.2) (end 144.5 96.4) (width 0.2) (layer "B.Cu") (net 27))
   (segment (start 171.25 99.5275) (end 171.25 101.17) (width 0.2) (layer "B.Cu") (net 27))
   (segment (start 152.1 93.6) (end 159.1 100.6) (width 0.2) (layer "B.Cu") (net 27))
@@
   (segment (start 161.7 101.88) (end 161.7 104.873) (width 0.2) (layer "F.Cu") (net 73))
   (segment (start 128.88 103.2514) (end 128.88 102.95) (width 0.2) (layer "F.Cu") (net 73))
-  (segment (start 169.5 98.57) (end 171.9 98.57) (width 1) (layer "F.Cu") (net 75))
-  (segment (start 170.7 98.57) (end 170.7 96.8875) (width 1) (layer "F.Cu") (net 75))
-  (segment (start 167.134 97.03) (end 167.754 97.65) (width 1) (layer "F.Cu") (net 75))
+  (segment (start 168.7 98.35) (end 169.0375 98.35) (width 1) (layer "F.Cu") (net 75))
+  (segment (start 170.6 98.47) (end 170.7 98.57) (width 0.25) (layer "F.Cu") (net 75))
   (segment (start 166.33 97.03) (end 166.33 97.65) (width 0.5) (layer "F.Cu") (net 75))
-  (segment (start 169.4672 98.6028) (end 169.5 98.57) (width 1) (layer "F.Cu") (net 75))
-  (segment (start 168.7068 98.6028) (end 169.4672 98.6028) (width 1) (layer "F.Cu") (net 75))
+  (segment (start 169.0375 98.35) (end 170.6 96.7875) (width 1) (layer "F.Cu") (net 75))
+  (segment (start 171.9 98.57) (end 171.9 98.0875) (width 0.5) (layer "F.Cu") (net 75))
+  (segment (start 169.5 98.57) (end 170.7 98.57) (width 0.5) (layer "F.Cu") (net 75))
+  (segment (start 171.9 98.0875) (end 170.6 96.7875) (width 0.5) (layer "F.Cu") (net 75))
   (segment (start 173.475 96.7875) (end 173.5 96.7625) (width 0.25) (layer "F.Cu") (net 75))
-  (segment (start 166.33 97.03) (end 167.134 97.03) (width 1) (layer "F.Cu") (net 75))
-  (segment (start 167.754 97.65) (end 168.7068 98.6028) (width 1) (layer "F.Cu") (net 75))
+  (segment (start 167.38 97.03) (end 168.7 98.35) (width 1) (layer "F.Cu") (net 75))
+  (segment (start 171.9 98.57) (end 170.7 98.57) (width 0.5) (layer "F.Cu") (net 75))
+  (segment (start 170.6 96.7875) (end 170.6 97.47) (width 0.25) (layer "F.Cu") (net 75))
+  (segment (start 166.33 97.03) (end 167.38 97.03) (width 1) (layer "F.Cu") (net 75))
   (segment (start 170.6 96.7875) (end 173.475 96.7875) (width 1) (layer "F.Cu") (net 75))
+  (segment (start 170.6 97.47) (end 169.5 98.57) (width 0.25) (layer "F.Cu") (net 75))
   (segment (start 170.7 96.8875) (end 170.6 96.7875) (width 0.25) (layer "F.Cu") (net 75))
+  (segment (start 170.6 96.7875) (end 170.6 98.47) (width 0.25) (layer "F.Cu") (net 75))
   (segment (start 166.33 96.55) (end 166.33 97.03) (width 0.5) (layer "F.Cu") (net 75))
   (segment (start 169.35 87.45) (end 170.29 87.45) (width 0.2) (layer "F.Cu") (net 76))
@@
   (via (at 161.0614 88.7222) (size 0.8) (drill 0.4) (layers "F.Cu" "B.Cu") (free) (net 78))
   (via (at 159.0548 91.2368) (size 0.8) (drill 0.4) (layers "F.Cu" "B.Cu") (free) (net 78))
-  (segment (start 157.105 92.425) (end 156.95 92.27) (width 0.2) (layer "B.Cu") (net 78))
   (segment (start 160.9578 92.2) (end 159.9946 91.2368) (width 0.2) (layer "B.Cu") (net 78))
   (segment (start 156.95 92.27) (end 155.8925 92.27) (width 0.2) (layer "B.Cu") (net 78))
@@
   (segment (start 154.51 94) (end 155.2 94) (width 0.2) (layer "B.Cu") (net 78))
   (segment (start 155.8925 92.27) (end 155.6625 92.5) (width 0.2) (layer "B.Cu") (net 78))
+  (segment (start 157.47 92.27) (end 156.95 92.27) (width 0.2) (layer "B.Cu") (net 78))
+  (segment (start 158.25 92.425) (end 157.625 92.425) (width 0.2) (layer "B.Cu") (net 78))
+  (segment (start 157.625 92.425) (end 157.47 92.27) (width 0.2) (layer "B.Cu") (net 78))
   (segment (start 161.5875 92.2) (end 160.9578 92.2) (width 0.2) (layer "B.Cu") (net 78))
   (segment (start 159.0548 91.2368) (end 159.0548 91.6798) (width 0.2) (layer "B.Cu") (net 78))
@@
   (segment (start 159.0548 91.6798) (end 159.8 92.425) (width 0.2) (layer "B.Cu") (net 78))
   (segment (start 160.6494 92.425) (end 160.9344 92.71) (width 0.2) (layer "B.Cu") (net 78))
-  (segment (start 161.5875 91.2) (end 161.8628 91.2) (width 0.1) (layer "B.Cu") (net 78))
   (segment (start 160.9344 92.71) (end 160.9444 92.7) (width 0.2) (layer "B.Cu") (net 78))
   (segment (start 155.2 94) (end 155.6625 93.5375) (width 0.2) (layer "B.Cu") (net 78))
@@
   (segment (start 172.695 95.78) (end 172.7125 95.7625) (width 0.2) (layer "B.Cu") (net 82))
   (segment (start 172.7125 103.9375) (end 168.1 108.55) (width 0.5) (layer "B.Cu") (net 82))
-  (segment (start 128.3208 104.1908) (end 128.3208 105.2092) (width 0.2) (layer "F.Cu") (net 83))
   (segment (start 126.7968 102.6668) (end 128.3208 104.1908) (width 0.2) (layer "F.Cu") (net 83))
   (segment (start 128.29 106.3444) (end 128.9558 107.0102) (width 0.2) (layer "F.Cu") (net 83))
   (segment (start 127.88 99.26) (end 127.88 97.345) (width 0.2) (layer "F.Cu") (net 83))
-  (segment (start 128.3208 105.2092) (end 128.29 105.24) (width 0.2) (layer "F.Cu") (net 83))
+  (segment (start 128.3208 104.1908) (end 128.3208 105.2092) (width 0.2) (layer "F.Cu") (net 83))
   (segment (start 127.054 99.26) (end 126.7968 99.5172) (width 0.2) (layer "F.Cu") (net 83))
   (segment (start 130.55 102.9) (end 130.55 102.0886) (width 0.25) (layer "F.Cu") (net 83))
@@
   (segment (start 126.7968 99.5172) (end 126.7968 102.6668) (width 0.2) (layer "F.Cu") (net 83))
   (segment (start 128.29 105.24) (end 128.29 106.3444) (width 0.2) (layer "F.Cu") (net 83))
-  (segment (start 128.29 105.24) (end 128.29 105.16) (width 0.25) (layer "F.Cu") (net 83))
+  (segment (start 128.3208 105.2092) (end 128.29 105.24) (width 0.2) (layer "F.Cu") (net 83))
   (segment (start 131.7498 102.8954) (end 130.943 102.0886) (width 0.2) (layer "F.Cu") (net 83))
   (segment (start 127.88 99.26) (end 127.054 99.26) (width 0.2) (layer "F.Cu") (net 83))
@@
       )
     )
-  )
-  (zone (net 78) (net_name "Net-(C1-Pad1)") (layer "B.Cu") (hatch edge 0.508)
-    (connect_pads yes (clearance 0.508))
-    (min_thickness 0.254) (filled_areas_thickness no)
-    (fill yes (thermal_gap 0.508) (thermal_bridge_width 0.508))
-    (polygon
-      (pts
-        (xy 161.8 92.8)
-        (xy 161.4 92.8)
-        (xy 160.25 92.7)
-        (xy 155.7 92.7)
-        (xy 155.7 92.1)
-        (xy 161.8 92.1)
-      )
-    )

Commit message: Routing complete
Parts:
- removed TP3, TP4, TP5, TP6: TestPoint, TestPoint:TestPoint_Pad_D1.0mm
- moved TP8 2.93 mm to (140.3, 94.7)
Connections:
- net GMS_STATUS_EXT renamed GMS_STATUS
- J3 pad 06: GSM_TXD_ESP_RTS -> GSM_RTS
- J3 pad 07: GSM_RXD_ESP_CTS -> GSM_CTS
- J3 pad 10: GSM_DTR_EXT -> unconnected-(J3-Pad10)
Routing:
- net GSM_CTS: track 3.14 -> 61.8 mm, vias 0 -> 2
- net GSM_RTS: track 3.47 -> 51.5 mm, vias 0 -> 2
- net GSM_DCD: track 5.02 -> 0.00 mm
- net GSM_DTR: track 3.33 -> 0.00 mm
- net GSM_STATUS: track 3.86 -> 2.33 mm
- net RTS: track 13.8 -> 12.5 mm
- net GND: vias 23 -> 24
Other:
- board size 54 x 28 mm -> 52 x 29 mm
